File: Science_Board/_restore_backup_2026-10-23T14-51-32-663/ManualControls.kicad_sch (KiCad schematic)
At the start: 46 parts, among them SW1 SW_Push, SW10 SW_Push, SW11 SW_Push, SW12 SW_SPDT, SW2 SW_Push, SW3 SW_Push, SW4 SW_Push, SW5 SW_Push, SW6 SW_Push, SW7 SW_Push, SW8 SW_Push, SW9 SW_Push

Commit message: fixed pwm driver and a connecter footprint
Changed lines of the file:
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@@
 	(text "Servo Buttons"
 		(exclude_from_sim no)
-		(at 122.428 193.294 0)
+		(at 120.396 179.07 0)
 		(effects
 			(font
